File: pcb/Launch pad.kicad_sch (KiCad schematic)
At the start: 13 parts, among them SW10 SW_Push, SW11 SW_Push, SW12 SW_Push, SW13 SW_Push, SW7 SW_Push, SW9 SW_Push, U1 XIAO-RP2040-DIP

Commit message: added firmware
Connections:
- net +5V: now also D1.3 (VDD), D10.3 (VDD), D2.3 (VDD), D7.3 (VDD), D8.3 (VDD), D9.3 (VDD); no longer D1.4 (DOUT), D10.4 (DOUT), D2.4 (DOUT), D7.4 (DOUT), D8.4 (DOUT), D9.4 (DOUT)
- net GND: now also D1.1 (VSS), D10.1 (VSS), D2.1 (VSS), D7.1 (VSS), D8.1 (VSS), D9.1 (VSS); no longer D1.2 (DIN), D10.2 (DIN), D2.2 (DIN), D7.2 (DIN), D8.2 (DIN), D9.2 (DIN)
- net at U1.5 (GPIO6/SDA): now also D7.2 (DIN); no longer D7.3 (VDD)
- new net: D1.2 (DIN), D10.4 (DOUT)
- new net: D1.4 (DOUT), D2.2 (DIN)
- new net: D10.2 (DIN), D9.4 (DOUT)
- new net: D8.4 (DOUT), D9.2 (DIN)
- new net: D7.4 (DOUT), D8.2 (DIN)
Other:
- moved on the sheet: D1, D10, D2, D7, D8, D9
